File: Philips 212 II.kicad_pcb (KiCad board)
At the start: 2 copper layers, 148.5 x 125.7 mm, 66 parts, among them J1 ~14V AC, J2 33, J3 OFF, J4 45, J5 PROG, J6 STOP, J7 MOTOR, Q1 IRF8707PBF, SW1 RST, U1 LM7809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

Commit message: attempt to make analytical PID paramns
Parts:
- removed C8: 0.1u, Capacitor_SMD:C_0805_2012Metric_Pad1.18x1.45mm_HandSolder
- removed D10: 1N4148, Diode_SMD:D_MELF_Handsoldering
- added D11: BAT46, Diode_THT:D_DO-35_SOD27_P7.62mm_Horizontal, B.Cu at (172.6, 119.6)
Routing:
- net /tacho: track 118.3 -> 115.3 mm
- net /SENSOR_GND: track 146.1 -> 145.1 mm
- net GND: track 427.8 -> 427.3 mm
