File: Philips 212 II.kicad_sch (KiCad schematic)
At the start: 71 parts, among them J1 ~14V AC, J2 33, J3 OFF, J4 45, J5 PROG, J6 STOP, J7 MOTOR, Q1 IRF8707PBF, SW1 RST, U1 LM7809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

Commit message: attempt to make analytical PID paramns
Parts:
- removed C8: 0.1u, Capacitor_SMD:C_0805_2012Metric_Pad1.18x1.45mm_HandSolder, symbol Device:C_Small
- removed D10: 1N4148, Diode_SMD:D_MELF_Handsoldering, symbol Diode:1N4148WS
- added D11: BAT46, Diode_THT:D_DO-35_SOD27_P7.62mm_Horizontal, symbol Device:D_Schottky_Small
- R13, R15, R17: value 2.2M -> 10M
Connections:
- net +5V: now also D11.1 (K)
- net at J5.4 (Pin_4): now also D11.2 (A)
Other:
- note added: "BROWN BLACK RED YELLOW"
- note removed: "MOTOR +"
- note removed: "MOTOR-"
- note removed: "TACH INPUT"
